File: AK4558EN_Breakout.brd (EAGLE design)
At the start: 35.6 x 33 mm, 35 parts, among them U1 AK4558QFN28

Commit message: update file name
Routing:
- net GND: track 7.86 -> 2.03 mm
Other:
- board text added: "CAD0"
- board text added: "CAD1"
- board text added: "CKS2"
- board text added: "H"
- board text added: "L"
- board text added: "PIN H L CKS2 MASTER SLAVE CAD0 I2C ADDR BIT0 CAD1 I2C ADDR BIT1"
Changed lines of the file:
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@@
 </layers>
 <board>
+<fusionsync huburn="a.cGVyc29uYWw6dWUyYjk1ZDQw" projecturn="a.cGVyc29uYWw6dWUyYjk1ZDQwIzIwMjAwNTE5Mjk5NzQyNjI2" f3durn="urn:adsk.wipprod:dm.lineage:i5jWOPUDTBmhmqd-RuE_7Q" pcbguid="02b62b20-da48-490f-8417-fce784ffbc98" lastpulledtime="" lastsyncedchangeguid="" latestrevisionid="6aa4b20e-750f-4c2c-8944-5adc49d9522d" lastsyncedrevisionid="6aa4b20e-750f-4c2c-8944-5adc49d9522d" lastboardhashguid="8d34301d-7b35-94d6-a56c-fb8b15d0f61f" lastpushedtime="2020-05-24T13:08:44Z" linktopcb3d="%12"/>
 <plain>
 <wire x1="0" y1="0" x2="35.56" y2="0" width="0" layer="20"/>
@@
 <text x="15.875" y="30.48" size="1.143" layer="22" font="vector" ratio="15" rot="MR0" align="center-right">AK4558EN Breakout
 Copyright(C) Cultr.camp</text>
+<text x="20.32" y="15.875" size="1.143" layer="22" font="vector" ratio="15" rot="MR0" align="center-right">CAD1</text>
+<text x="20.32" y="13.843" size="1.143" layer="22" font="vector" ratio="15" rot="MR0" align="center-right">CAD0</text>
+<text x="18.415" y="15.875" size="1.143" layer="22" font="vector" ratio="15" rot="MR0" align="center">H</text>
+<text x="15.4178" y="15.875" size="1.143" layer="22" font="vector" ratio="15" rot="MR0" align="center">L</text>
+<wire x1="13.9446" y1="16.8656" x2="13.9446" y2="14.859" width="0.1524" layer="22"/>
+<wire x1="13.9446" y1="14.859" x2="13.9446" y2="12.8778" width="0.1524" layer="22"/>
+<wire x1="13.9446" y1="12.8778" x2="19.8882" y2="12.8778" width="0.1524" layer="22"/>
+<wire x1="19.8882" y1="12.8778" x2="19.8882" y2="14.859" width="0.1524" layer="22"/>
+<wire x1="19.8882" y1="14.859" x2="19.8882" y2="16.8656" width="0.1524" layer="22"/>
+<wire x1="19.8882" y1="16.8656" x2="13.9446" y2="16.8656" width="0.1524" layer="22"/>
+<text x="18.415" y="13.843" size="1.143" layer="22" font="vector" ratio="15" rot="MR0" align="center">H</text>
+<text x="15.4178" y="13.843" size="1.143" layer="22" font="vector" ratio="15" rot="MR0" align="center">L</text>
+<wire x1="13.9446" y1="14.859" x2="19.8882" y2="14.859" width="0.1524" layer="22"/>
+<text x="18.8722" y="26.67" size="1.143" layer="22" font="vector" ratio="15" rot="MR0" align="center">H</text>
+<text x="15.875" y="26.67" size="1.143" layer="22" font="vector" ratio="15" rot="MR0" align="center">L</text>
+<wire x1="14.4526" y1="27.6606" x2="14.4526" y2="25.7048" width="0.1524" layer="22"/>
+<wire x1="14.4526" y1="25.7048" x2="20.3454" y2="25.7048" width="0.1524" layer="22"/>
+<wire x1="20.3454" y1="25.7048" x2="20.3454" y2="27.6606" width="0.1524" layer="22"/>
+<wire x1="20.3454" y1="27.6606" x2="14.4526" y2="27.6606" width="0.1524" layer="22"/>
+<text x="20.574" y="26.67" size="1.143" layer="22" font="vector" ratio="15" rot="MR0" align="center-right">CKS2</text>
+<text x="27.94" y="4.445" size="0.889" layer="22" font="vector" ratio="15" rot="MR0" align="center-left">PIN          H           L
+CKS2  MASTER  SLAVE
+CAD0 I2C ADDR BIT0
+CAD1 I2C ADDR BIT1</text>
 </plain>
 <attributes>
@@
 <vertex x="35.56" y="0"/>
 </polygon>
-<wire x1="17.51" y1="19.09" x2="17.51" y2="19.6502" width="0.1524" layer="1"/>
-<wire x1="17.4752" y1="19.685" x2="16.51" y2="19.685" width="0.1524" layer="1"/>
-<wire x1="17.51" y1="19.6502" x2="17.4752" y2="19.685" width="0.1524" layer="1"/>
-<wire x1="17.51" y1="19.6502" x2="17.5284" y2="19.6686" width="0.1524" layer="1"/>
-<wire x1="17.5284" y1="19.6686" x2="18.0594" y2="19.6686" width="0.1524" layer="1"/>
-<wire x1="16.51" y1="19.685" x2="16.51" y2="21.51" width="0.1524" layer="1"/>
 <wire x1="16.51" y1="21.51" x2="16.55" y2="21.55" width="0.1524" layer="1"/>
-<wire x1="19.01" y1="21.59" x2="18.415" y2="21.59" width="0.2032" layer="1"/>
-<wire x1="18.415" y1="21.59" x2="18.415" y2="21.3192125" width="0.2032" layer="1"/>
-<wire x1="18.415" y1="21.3192125" x2="18.406" y2="21.3102125" width="0.2032" layer="1"/>
-<wire x1="18.406" y1="21.3102125" x2="18.406" y2="20.955" width="0.2032" layer="1"/>
-<wire x1="18.415" y1="21.59" x2="18.415" y2="21.8607875" width="0.2032" layer="1"/>
-<wire x1="18.415" y1="21.8607875" x2="18.406" y2="21.8697875" width="0.2032" layer="1"/>
-<wire x1="18.406" y1="21.8697875" x2="18.406" y2="22.225" width="0.2032" layer="1"/>
 <via x="17.8054" y="17.6022" extent="1-16" drill="0.35"/>
 <via x="17.145" y="11.43" extent="1-16" drill="0.35"/>
@@
 <contactref element="I2C" pad="5"/>
 <contactref element="R15" pad="2"/>
-<wire x1="17.01" y1="24.09" x2="17.01" y2="25.4" width="0.1524" layer="1"/>
-<wire x1="19.7222" y1="26.0722" x2="19.7222" y2="26.67" width="0.1524" layer="1"/>
-<wire x1="17.01" y1="25.4" x2="17.145" y2="25.4" width="0.1524" layer="1"/>
-<wire x1="17.145" y1="25.4" x2="19.05" y2="25.4" width="0.1524" layer="1"/>
-<wire x1="19.05" y1="25.4" x2="19.7222" y2="26.0722" width="0.1524" layer="1"/>
 <wire x1="1.905" y1="3.175" x2="1.905" y2="7.5198" width="0.4064" layer="1"/>
 <wire x1="1.905" y1="7.5198" x2="2.0052" y2="7.62" width="0.4064" layer="1"/>
@@
 <wire x1="18.415" y1="10.795" x2="18.415" y2="6.9596" width="0.2032" layer="1"/>
 <wire x1="19.265" y1="11.645" x2="18.415" y2="10.795" width="0.2032" layer="1"/>
-<via x="17.145" y="25.4" extent="1-16" drill="0.35"/>
 <wire x1="11.43" y1="25.4" x2="10.795" y2="24.765" width="0.2032" layer="16"/>
 <wire x1="10.795" y1="24.765" x2="10.795" y2="20.32" width="0.2032" layer="16"/>
-<wire x1="17.145" y1="25.4" x2="11.43" y2="25.4" width="0.2032" layer="16"/>
+<wire x1="17.01" y1="24.09" x2="17.01" y2="24.9856" width="0.2032" layer="1"/>
+<wire x1="17.01" y1="24.9856" x2="17.3482" y2="25.3238" width="0.2032" layer="1"/>
+<via x="17.3482" y="25.3238" extent="1-16" drill="0.35"/>
+<wire x1="17.3482" y1="25.3238" x2="14.6812" y2="25.3238" width="0.2032" layer="16"/>
+<wire x1="14.6812" y1="25.3238" x2="14.605" y2="25.4" width="0.2032" layer="16"/>
+<wire x1="14.605" y1="25.4" x2="11.43" y2="25.4" width="0.2032" layer="16"/>
+<wire x1="17.3482" y1="25.3238" x2="17.4244" y2="25.4" width="0.2032" layer="1"/>
+<wire x1="19.7222" y1="25.7674" x2="19.7222" y2="26.67" width="0.2032" layer="1"/>
+<wire x1="17.4244" y1="25.4" x2="19.3548" y2="25.4" width="0.2032" layer="1"/>
+<wire x1="19.3548" y1="25.4" x2="19.7222" y2="25.7674" width="0.2032" layer="1"/>
 </signal>
 <signal name="SDO">
@@
 </note>
 <note version="8.3" severity="warning">
+Since Version 8.3, EAGLE supports Fusion synchronisation.
+This feature will not be available in this version and saving
+the document will break the link to the Fusion PCB feature.
+</note>
+<note version="8.3" severity="warning">

Commit message: update schematic and add gerber
Parts:
- moved AUDIO 15.2 mm to (32.7, 24.1), turned to 270 degrees
Connections:
- net BCK renamed N$12
- net LRCK renamed N$14
- net SDI renamed N$13
- net SDO renamed N$1
- net GND: now also I2C.5; no longer I2C.4
- net LIN: now also AUDIO.7; no longer AUDIO.1
- net LOUT: now also AUDIO.3; no longer AUDIO.5
- net RIN: now also AUDIO.5; no longer AUDIO.3
- net ROUT: now also AUDIO.1; no longer AUDIO.7
- net VCC: now also I2C.4; no longer I2C.5
Routing:
- net GND: track 2.03 -> 5.17 mm, vias 53 -> 50
- net CODEC_AVDD: track 22.6 -> 25.5 mm
- net N$7: track 10.1 -> 8.08 mm, vias 0 -> 2
- net VCC: track 80.5 -> 82.3 mm
- net N$2: track 15.8 -> 17.1 mm
- net N$6: track 13.1 -> 12.2 mm
- net PDN: track 29.6 -> 30.5 mm
